File: business-card/businesscard_a1/businesscard_a1.kicad_pcb (KiCad board)
At the start: 2 copper layers, 85.8 x 54.2 mm, 12 parts, among them P1 NFC, P2 CREDIT_CARD, U1 NTAG_NT3H1X01

Commit message: Add OSHW logo
Parts:
- added G***: OSHWMASK5MM, business-card:OSHWMASK5MM, B.Cu at (184.0, 118.0)

Commit message: Reconnect chip
Parts:
- removed the G*** at (184.0, 118.0)
- C1: value C -> 220n
- P1: footprint Pin_Headers:Pin_Header_Straight_1x02 -> business-card:BUSINESS_NFC_ANTENNA_4X5CM; moved to B.Cu
- moved P1 64.7 mm to (168.5, 97.0), turned to 90 degrees
- moved R1 5.10 mm to (120.0, 96.1)
- moved U1 3.80 mm to (120.0, 91.4), turned to 270 degrees
- moved D1 2.90 mm to (120.0, 94.9)
- moved C1 0.70 mm to (120.0, 93.7), turned to 180 degrees
- moved G*** 0.40 mm to (145.3, 89.3)
Connections:
- C1 pad 1: Net-(C1-Pad1) -> VDD
- D1 pad 1: GND -> Net-(D1-Pad1)
- D1 pad 2: Net-(D1-Pad2) -> VDD
- P1 pad 1: Net-(P1-Pad1) -> /LB
- P1 pad 2: Net-(P1-Pad2) -> /LA
- P2 pad C1: Net-(P2-PadC1) -> /SCL
- P2 pad C2: (no net) -> /FIELD
- P2 pad C3: (no net) -> /SDA
- P2 pad C4: Net-(P2-PadC4) -> GND
- P2 pad C5: Net-(P2-PadC5) -> /LA
- P2 pad C6: (no net) -> /LB
- P2 pad C7: (no net) -> VDD
- R1 pad 1: Net-(R1-Pad1) -> Net-(D1-Pad1)
- R1 pad 2: Net-(D1-Pad2) -> GND
- U1 pad 1: Net-(P1-Pad1) -> /LA
- U1 pad 3: (no net) -> /SCL
- U1 pad 4: (no net) -> /FIELD
- U1 pad 5: (no net) -> /SDA
- U1 pad 6: Net-(C1-Pad1) -> VDD
- U1 pad 7: Net-(R1-Pad1) -> VDD
- U1 pad 8: Net-(P1-Pad2) -> /LB
Routing:
- net /LA: track 0.00 -> 57.3 mm, vias 0 -> 1
- net /LB: track 0.00 -> 53.1 mm, vias 0 -> 1
- net GND: track 0.00 -> 13.2 mm, vias 0 -> 2
- net /SCL: track 0.00 -> 9.01 mm
- net VDD: track 0.00 -> 7.70 mm
- net /SDA: track 0.00 -> 6.64 mm
- net /FIELD: track 0.00 -> 3.77 mm
- net Net-(P2-PadC8): track 0.00 -> 3.21 mm
- net Net-(D1-Pad1): track 0.00 -> 1.68 mm
Other:
- net class Default: trace_width 0.25 -> 0.2; via_dia 0.6 -> 0.7

Commit message: Small mods
Parts:
- P1: footprint business-card:BUSINESS_NFC_ANTENNA_4X5CM -> business-card:BUSINESS_NFC_ANTENNA_4X5CM_NEW
- moved P1 0.10 mm to (168.5, 97.1)
Routing:
- net /LA: track 57.3 -> 37.6 mm
- net /LB: track 53.1 -> 34.0 mm
Other:
- board size 85.8 x 54.2 mm -> 85.6 x 54 mm
- net class Default: via_drill 0.4 -> 0.3
- rule pad_to_mask_clearance: 0.15 -> 0.1
- rule solder_mask_min_width: 0.15 -> 0.1
